File: miniusbradiointerface.sch (KiCad schematic (older format))
At the start: 22 parts, among them J1 VCC, J2 DP, J3 DM, J4 GND, J5 DB9_Male, Q1 BSS138, U1 CM108AH, Y1 12M

Commit message: Properly archived symbols
Parts:
- U1: symbol Cmedia_USB_Audio:CM108AH -> archive:Cmedia_USB_Audio_CM108AH
Changed lines of the file:
@@
 $EndDescr
 $Comp
-L Cmedia_USB_Audio:CM108AH U1
+L archive:Cmedia_USB_Audio_CM108AH U1
 U 1 1 5E75E071
 P 5100 3300
